File: SW9E-MSBv3.0.kicad_pcb (KiCad board)
At the start: 2 copper layers, 39.1 x 40.6 mm, 26 parts, among them J1 22-05-3021, J2 22-05-3021, J3 90120-0763, J4 90120-0763, J5 22-05-3021, P1 22-27-2041, P2 22-27-2041, P3 61300811121, Q1 FDN5632N-F085, Q2 FDN5632N-F085, U1 MSP430FR2355TPTR, U2 LD1117S33TR

Commit message: Stuff
Parts:
- removed C1: 100pF, AltiumImport:SMD-0805C
- removed C2: 10µF, AltiumImport:SMD-0805C
- removed D1: 1.9V, AltiumImport:FP-150080SS75000-MFG
- removed J5: 22-05-3021, AltiumImport:FP-22-05-3021-MFG
- removed P1, P2: 22-27-2041, AltiumImport:MOLX-22-27-2041_V
- removed P3: 61300811121, AltiumImport:61300811121
- removed R10: 0.0, AltiumImport:SMD-0805-RES
- removed R7: 309, AltiumImport:SMD-0805-RES
- removed U2: LD1117S33TR, AltiumImport:SOT-223_L
- added J6: SSW-104-03-F-S, Library:CON4_1X4_TU_SSQ, F.Cu at (127.0, 63.5)
- added J7: SSW-104-03-F-S, Library:CON4_1X4_TU_SSQ, F.Cu at (127.0, 76.2)
- moved G*** 49.5 mm to (109.3, 57.6)
- moved J3 16.2 mm to (147.1, 103.7)
- moved J4 16.2 mm to (147.1, 112.6)
- moved D3 16.2 mm to (120.2, 104.5)
- moved R9 16.2 mm to (126.3, 103.2)
- moved J2 16.2 mm to (151.4, 91.8)
- moved R1 16.2 mm to (138.7, 91.8)
- moved U1 16.2 mm to (131.1, 94.8)
- moved D2 16.2 mm to (142.0, 110.6)
- moved J1 16.2 mm to (151.4, 82.7)
- moved Q1 16.2 mm to (142.8, 93.8)
- moved Q2 16.2 mm to (142.8, 100.4)
- moved R2 16.2 mm to (138.7, 98.9)
- moved R3 16.2 mm to (138.7, 95.4)
- moved R4 16.2 mm to (138.7, 102.5)
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Connections:
- net +3V3 renamed +3.3V
- net +5 renamed +5V
Routing:
- net (no net): track 0.00 -> 29.0 mm, vias 0 -> 1
- net +3.3V: track 31.6 -> 16.7 mm
- net +5V: track 84.3 -> 77.6 mm, vias 1 -> 0
- net Net-(C2-Pad1): track 5.10 -> 0.00 mm
- net Net-(D1-A): track 2.30 -> 0.00 mm
- net GND: vias 5 -> 6
- added copper zone on F.Cu, net (none)
- removed copper zone on F.Cu, net Net-(C2-Pad1)
Other:
- board size 39.1 x 40.6 mm -> 105.5 x 93 mm
- board text added: "v3.0"
- board text removed: "v1.0"

Commit message: Stuff
Parts:
- added J5: 640453-8, Library:TE_640453-8, F.Cu at (86.7, 88.1)
- moved J7 57.9 mm to (127.0, 134.1)
- moved J3 30.4 mm to (175.8, 93.7), turned to -90 degrees
- moved J4 30.0 mm to (175.8, 103.9), turned to -90 degrees
- moved J1 25.2 mm to (175.8, 76.4)
- moved J2 25.2 mm to (175.8, 85.6)
- moved R8 10.3 mm to (132.1, 105.4), turned to -90 degrees
- moved D2 10.3 mm to (132.1, 107.9)
- moved R9 6.25 mm to (120.2, 101.8), turned to -90 degrees
- moved D3 2.04 mm to (122.2, 104.3), turned to 180 degrees
Routing:
- net +5V: track 77.6 -> 0.00 mm
- net /TXD: track 23.9 -> 69.4 mm, vias 0 -> 2
- net /RXD: track 22.1 -> 52.6 mm
- net (no net): track 29.0 -> 0.00 mm, vias 1 -> 0
- net /SERVO1_CTRL: track 20.5 -> 49.4 mm
- net /SERVO2_CTRL: track 21.0 -> 47.9 mm, vias 2 -> 0
- net /SDA: track 23.8 -> 0.00 mm
- net Net-(Q2-D): track 11.6 -> 34.9 mm
- net /TST: track 24.0 -> 45.3 mm
- net Net-(Q1-D): track 14.2 -> 35.3 mm
- net /SCL: track 21.2 -> 0.55 mm
- net /RST: track 23.9 -> 40.6 mm
- net Net-(U1-P6.2/TB3.3): track 14.1 -> 6.82 mm, vias 2 -> 0
- net +3.3V: track 16.7 -> 11.7 mm, vias 1 -> 0
- net Net-(D3-A): track 5.02 -> 2.53 mm, vias 2 -> 0
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