File: SW9E-MSBv3.0.kicad_sch (KiCad schematic)
At the start: 25 parts, among them J1 22-05-3021, J2 22-05-3021, J3 90120-0763, J4 90120-0763, J5 22-05-3021, P1 22-27-2041, P2 22-27-2041, P3 61300811121, Q1 FDN5632N-F085, Q2 FDN5632N-F085, U1 MSP430FR2355TPTR, U2 LD1117S33TR

Commit message: Stuff
Parts:
- removed C1: 100pF, AltiumImport:SMD-0805C, symbol MSB-altium-import:root_0_GQM2195C1H101JB01D
- removed C2: 10µF, AltiumImport:SMD-0805C, symbol MSB-altium-import:root_0_GCJ21BR71A106KE01L
- removed D1: 1.9V, AltiumImport:FP-150080SS75000-MFG, symbol MSB-altium-import:root_0_8706943c75ba83719d021d2fdc84c58
- removed J5: 22-05-3021, AltiumImport:FP-22-05-3021-MFG, symbol MSB-altium-import:root_0_3bc925449376181038e59eaffc5286c
- removed P1, P2: 22-27-2041, AltiumImport:MOLX-22-27-2041_V, symbol MSB-altium-import:root_2_CN-1P-M-R4
- removed P3: 61300811121, AltiumImport:61300811121, symbol MSB-altium-import:root_0_WE-CN-1P-M-R8
- removed R10: 0.0, AltiumImport:SMD-0805-RES, symbol MSB-altium-import:root_1_ERJ-6GEY0R00V
- removed R7: 309, AltiumImport:SMD-0805-RES, symbol MSB-altium-import:root_1_ERJ-6ENF3090V
- removed U2: LD1117S33TR, AltiumImport:SOT-223_L, symbol MSB-altium-import:root_0_PM-REG-LD1117-SOT4
- added J3, J4: SSW-104-03-F-S, CON4_1X4_TU_SSQ, symbol 2024-01-30_02-53-16:SSW-104-03-F-S
- added J5: 640453-8, 640453-8:TE_640453-8, symbol New_Library:640453-8
Connections:
- net GND: now also J3.1, J5.8
- net RST: now also J5.5
- net RXD: now also J5.3
- net SCL: now also J4.1
- net SDA: now also J4.2
- net TST: now also J5.6
- net TXD: now also J5.4
- net +3V3 renamed +3.3V
- net +3.3V: now also J3.2
- net +5 renamed +5V
- net +5V: now also J3.3, J5.7
- new net +12V: J3.4
- no-connect marks 0 -> 2
Other:
- note removed: "5Vin Header"
- note removed: "Chain Header"
- note removed: "I2C Daisy"

Commit message: Stuff
Parts:
- J3, J4: footprint AltiumImport:FP-90120-0763-MFG -> CONN_901200763_MOL; symbol MSB-altium-import:root_0_0d3f023dd272f625e17a2be33dea85f -> 2024-02-03_17-19-22:901200763
- J5: footprint 640453-8:TE_640453-8 -> Library:TE_640453-8
Connections:
- net +5V: now also J5.A5; no longer J5.7
- net GND: now also J3.3, J4.3, J5.A6; no longer J3.2, J4.2, J5.8
- net RST: now also J5.A3; no longer J5.5
- net RXD: now also J5.A1; no longer J5.3
- net SERVO1_CTRL: now also J3.2; no longer J3.3
- net SERVO2_CTRL: now also J4.2; no longer J4.3
- net TST: now also J5.A4; no longer J5.6
- net TXD: now also J5.A2; no longer J5.4
- no-connect marks 2 -> 40
