File: MSB.kicad_sch (KiCad schematic)
At the start: 25 parts, among them J1 22-05-3021, J2 22-05-3021, J3 90120-0763, J4 90120-0763, J5 22-05-3021, P1 22-27-2041, P2 22-27-2041, P3 61300811121, Q1 FDN5632N-F085, Q2 FDN5632N-F085, U1 MSP430FR2355TPTR, U2 LD1117S33TR

Commit message: Fix footprint linking and logos
Parts:
- C1: value ${ALTIUM_VALUE} -> 100pF; footprint SMD-0805C -> AltiumImport:SMD-0805C
- C2: value ${ALTIUM_VALUE} -> 10µF; footprint SMD-0805C -> AltiumImport:SMD-0805C
- D1, D3: footprint FP-150080SS75000-MFG -> AltiumImport:FP-150080SS75000-MFG
- D2: footprint FP-LTST-C171GKT-MFG -> AltiumImport:FP-LTST-C171GKT-MFG
- J1, J2, J5: footprint FP-22-05-3021-MFG -> AltiumImport:FP-22-05-3021-MFG
- J3, J4: footprint FP-90120-0763-MFG -> AltiumImport:FP-90120-0763-MFG
- P1, P2: footprint MOLX-22-27-2041_V -> AltiumImport:MOLX-22-27-2041_V
- P3: footprint 61300811121 -> AltiumImport:61300811121
- Q1, Q2: footprint SOT95P237X122-3N -> AltiumImport:SOT95P237X122-3N
- R1, R2: value ${ALTIUM_VALUE} -> 200; footprint SMD-0805-RES -> AltiumImport:SMD-0805-RES
- R10: value ${ALTIUM_VALUE} -> 0.0; footprint SMD-0805-RES -> AltiumImport:SMD-0805-RES
- R3, R4: value ${ALTIUM_VALUE} -> 10k; footprint SMD-0805-RES -> AltiumImport:SMD-0805-RES
- R7: value ${ALTIUM_VALUE} -> 309; footprint SMD-0805-RES -> AltiumImport:SMD-0805-RES
- R8: value ${ALTIUM_VALUE} -> 76.8; footprint SMD-0805-RES -> AltiumImport:SMD-0805-RES
- R9: value ${ALTIUM_VALUE} -> 140; footprint SMD-0805-RES -> AltiumImport:SMD-0805-RES
- U1: footprint FP-PT0048A-MFG -> AltiumImport:FP-PT0048A-MFG
- U2: footprint SOT-223_L -> AltiumImport:SOT-223_L
Changed lines of the file:
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@@
       (effects (font (size 1.27 1.27)) (justify left bottom))
     )
-    (property "Footprint" "SOT-223_L" (at 203.2 53.34 0)
+    (property "Footprint" "AltiumImport:SOT-223_L" (at 203.2 53.34 0)
       (effects (font (size 1.27 1.27)) hide)
     )
@@
       (effects (font (size 1.27 1.27)) (justify left bottom))
     )
-    (property "Footprint" "FP-LTST-C171GKT-MFG" (at 208.28 160.02 0)
+    (property "Footprint" "AltiumImport:FP-LTST-C171GKT-MFG" (at 208.28 160.02 0)
       (effects (font (size 1.27 1.27)) hide)
     )
@@
       (effects (font (size 1.27 1.27)) (justify left bottom))
     )
-    (property "Value" "${ALTIUM_VALUE}" (at 226.822 50.546 0)
-      (effects (font (size 1.27 1.27)) (justify left bottom))
-    )
-    (property "Footprint" "SMD-0805-RES" (at 226.06 48.26 0)
+    (property "Value" "0.0" (at 226.822 50.546 0)
+      (effects (font (size 1.27 1.27)) (justify left bottom))
+    )
+    (property "Footprint" "AltiumImport:SMD-0805-RES" (at 226.06 48.26 0)
       (effects (font (size 1.27 1.27)) hide)
     )
@@
       (effects (font (size 1.27 1.27)) (justify left bottom))
     )
-    (property "Footprint" "SOT95P237X122-3N" (at 58.42 43.18 0)
+    (property "Footprint" "AltiumImport:SOT95P237X122-3N" (at 58.42 43.18 0)
       (effects (font (size 1.27 1.27)) hide)
     )
@@
       (effects (font (size 1.27 1.27)) (justify left bottom))
     )
-    (property "Footprint" "FP-150080SS75000-MFG" (at 220.98 160.02 0)
+    (property "Footprint" "AltiumImport:FP-150080SS75000-MFG" (at 220.98 160.02 0)
       (effects (font (size 1.27 1.27)) hide)
     )
@@
       (effects (font (size 1.27 1.27)) (justify left bottom))
     )
-    (property "Value" "${ALTIUM_VALUE}" (at 27.686 74.422 0)
-      (effects (font (size 1.27 1.27)) (justify left bottom))
-    )
-    (property "Footprint" "SMD-0805-RES" (at 30.48 71.12 0)
+    (property "Value" "200" (at 27.686 74.422 0)
+      (effects (font (size 1.27 1.27)) (justify left bottom))
+    )
+    (property "Footprint" "AltiumImport:SMD-0805-RES" (at 30.48 71.12 0)
       (effects (font (size 1.27 1.27)) hide)
     )
@@
       (effects (font (size 1.27 1.27)) (justify left bottom))
     )
-    (property "Footprint" "FP-22-05-3021-MFG" (at 83.82 50.8 0)
+    (property "Footprint" "AltiumImport:FP-22-05-3021-MFG" (at 83.82 50.8 0)
       (effects (font (size 1.27 1.27)) hide)
     )
@@
       (effects (font (size 1.27 1.27)) (justify left bottom))
     )
-    (property "Footprint" "MOLX-22-27-2041_V" (at 15.24 121.92 0)
+    (property "Footprint" "AltiumImport:MOLX-22-27-2041_V" (at 15.24 121.92 0)
       (effects (font (size 1.27 1.27)) hide)
     )
@@
       (effects (font (size 1.27 1.27)) (justify left bottom))
     )
-    (property "Footprint" "61300811121" (at 220.98 99.06 0)
+    (property "Footprint" "AltiumImport:61300811121" (at 220.98 99.06 0)
       (effects (font (size 1.27 1.27)) hide)
     )
@@
       (effects (font (size 1.27 1.27)) (justify left bottom))
     )
-    (property "Footprint" "SOT95P237X122-3N" (at 58.42 73.66 0)
+    (property "Footprint" "AltiumImport:SOT95P237X122-3N" (at 58.42 73.66 0)
       (effects (font (size 1.27 1.27)) hide)
     )
@@
       (effects (font (size 1.27 1.27)) (justify left bottom))
     )
-    (property "Footprint" "FP-90120-0763-MFG" (at 134.62 76.2 0)
+    (property "Footprint" "AltiumImport:FP-90120-0763-MFG" (at 134.62 76.2 0)
       (effects (font (size 1.27 1.27)) hide)
     )
@@
       (effects (font (size 1.27 1.27)) (justify left bottom))
     )
-    (property "Value" "${ALTIUM_VALUE}" (at 197.104 68.326 0)
-      (effects (font (size 1.27 1.27)) (justify left bottom))
-    )
-    (property "Footprint" "SMD-0805C" (at 195.58 66.04 0)
+    (property "Value" "100pF" (at 197.104 68.326 0)
+      (effects (font (size 1.27 1.27)) (justify left bottom))
+    )
+    (property "Footprint" "AltiumImport:SMD-0805C" (at 195.58 66.04 0)
       (effects (font (size 1.27 1.27)) hide)
     )
@@
       (effects (font (size 1.27 1.27)) (justify left bottom))
     )
-    (property "Footprint" "FP-90120-0763-MFG" (at 134.62 43.18 0)
+    (property "Footprint" "AltiumImport:FP-90120-0763-MFG" (at 134.62 43.18 0)
       (effects (font (size 1.27 1.27)) hide)
     )
@@
       (effects (font (size 1.27 1.27)) (justify left bottom))
     )
-    (property "Value" "${ALTIUM_VALUE}" (at 200.914 160.274 0)
-      (effects (font (size 1.27 1.27)) (justify left bottom))
-    )
-    (property "Footprint" "SMD-0805-RES" (at 200.66 157.48 0)
+    (property "Value" "76.8" (at 200.914 160.274 0)
+      (effects (font (size 1.27 1.27)) (justify left bottom))
+    )
+    (property "Footprint" "AltiumImport:SMD-0805-RES" (at 200.66 157.48 0)
       (effects (font (size 1.27 1.27)) hide)
     )
@@
       (effects (font (size 1.27 1.27)) (justify left bottom))
     )
-    (property "Footprint" "FP-PT0048A-MFG" (at 35.56 104.14 0)
+    (property "Footprint" "AltiumImport:FP-PT0048A-MFG" (at 35.56 104.14 0)
       (effects (font (size 1.27 1.27)) hide)
     )
@@
       (effects (font (size 1.27 1.27)) (justify left bottom))
     )
-    (property "Value" "${ALTIUM_VALUE}" (at 221.742 154.686 0)
-      (effects (font (size 1.27 1.27)) (justify left bottom))
-    )
-    (property "Footprint" "SMD-0805-RES" (at 220.98 152.4 0)
+    (property "Value" "140" (at 221.742 154.686 0)
+      (effects (font (size 1.27 1.27)) (justify left bottom))
+    )
+    (property "Footprint" "AltiumImport:SMD-0805-RES" (at 220.98 152.4 0)
       (effects (font (size 1.27 1.27)) hide)
     )
@@
       (effects (font (size 1.27 1.27)) (justify left bottom))
     )
-    (property "Footprint" "FP-22-05-3021-MFG" (at 180.34 55.88 0)
+    (property "Footprint" "AltiumImport:FP-22-05-3021-MFG" (at 180.34 55.88 0)
       (effects (font (size 1.27 1.27)) hide)
     )
@@
       (effects (font (size 1.27 1.27)) (justify left bottom))
     )
-    (property "Value" "${ALTIUM_VALUE}" (at 38.862 50.546 0)
-      (effects (font (size 1.27 1.27)) (justify left bottom))
-    )
-    (property "Footprint" "SMD-0805-RES" (at 38.1 48.26 0)
+    (property "Value" "10k" (at 38.862 50.546 0)
+      (effects (font (size 1.27 1.27)) (justify left bottom))
+    )
+    (property "Footprint" "AltiumImport:SMD-0805-RES" (at 38.1 48.26 0)
       (effects (font (size 1.27 1.27)) hide)
     )
@@
       (effects (font (size 1.27 1.27)) (justify left bottom))
     )
-    (property "Value" "${ALTIUM_VALUE}" (at 227.584 68.326 0)
-      (effects (font (size 1.27 1.27)) (justify left bottom))
-    )
-    (property "Footprint" "SMD-0805C" (at 226.06 66.04 0)
+    (property "Value" "10µF" (at 227.584 68.326 0)
+      (effects (font (size 1.27 1.27)) (justify left bottom))
+    )
+    (property "Footprint" "AltiumImport:SMD-0805C" (at 226.06 66.04 0)
       (effects (font (size 1.27 1.27)) hide)
     )
@@
       (effects (font (size 1.27 1.27)) (justify left bottom))
     )
-    (property "Value" "${ALTIUM_VALUE}" (at 183.642 73.406 0)
-      (effects (font (size 1.27 1.27)) (justify left bottom))
-    )
-    (property "Footprint" "SMD-0805-RES" (at 182.88 71.12 0)
+    (property "Value" "309" (at 183.642 73.406 0)
+      (effects (font (size 1.27 1.27)) (justify left bottom))
+    )
+    (property "Footprint" "AltiumImport:SMD-0805-RES" (at 182.88 71.12 0)
       (effects (font (size 1.27 1.27)) hide)
     )
@@
       (effects (font (size 1.27 1.27)) (justify left bottom))
     )
-    (property "Footprint" "FP-150080SS75000-MFG" (at 185.42 83.82 0)
+    (property "Footprint" "AltiumImport:FP-150080SS75000-MFG" (at 185.42 83.82 0)
       (effects (font (size 1.27 1.27)) hide)
     )
@@
       (effects (font (size 1.27 1.27)) (justify left bottom))
     )
-    (property "Value" "${ALTIUM_VALUE}" (at 38.862 81.026 0)
-      (effects (font (size 1.27 1.27)) (justify left bottom))
-    )
-    (property "Footprint" "SMD-0805-RES" (at 38.1 78.74 0)
+    (property "Value" "10k" (at 38.862 81.026 0)
+      (effects (font (size 1.27 1.27)) (justify left bottom))
+    )
+    (property "Footprint" "AltiumImport:SMD-0805-RES" (at 38.1 78.74 0)
       (effects (font (size 1.27 1.27)) hide)
     )
@@
       (effects (font (size 1.27 1.27)) (justify left bottom))
     )
-    (property "Footprint" "MOLX-22-27-2041_V" (at 17.78 195.58 0)
+    (property "Footprint" "AltiumImport:MOLX-22-27-2041_V" (at 17.78 195.58 0)
       (effects (font (size 1.27 1.27)) hide)
     )
@@
       (effects (font (size 1.27 1.27)) (justify left bottom))
     )
-    (property "Footprint" "FP-22-05-3021-MFG" (at 83.82 81.28 0)
+    (property "Footprint" "AltiumImport:FP-22-05-3021-MFG" (at 83.82 81.28 0)
       (effects (font (size 1.27 1.27)) hide)
     )
@@
       (effects (font (size 1.27 1.27)) (justify left bottom))
     )
-    (property "Value" "${ALTIUM_VALUE}" (at 27.686 43.942 0)
-      (effects (font (size 1.27 1.27)) (justify left bottom))
-    )
-    (property "Footprint" "SMD-0805-RES" (at 30.48 40.64 0)
-      (effects (font (size 1.27 1.27)) hide)
-    )
+    (property "Value" "200" (at 27.686 43.942 0)
+      (effects (font (size 1.27 1.27)) (justify left bottom))
+    )
+    (property "Footprint" "AltiumImport:SMD-0805-RES" (at 30.48 40.64 0)
+      (effects (font (size 1.27 1.27)) hide)
+    )

Commit message: Cleanup sumbol field table
Parts:
- C1: DATASHEET URL http://www.murata.com/~/media/webrenewal/support/library/ca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 -> (none); MANUFACTURER Murata Electronics North America -> (none); MANUFACTURER PART NUMBER GQM2195C1H101JB01D -> (none); MOUNT Surface Mount, MLCC -> (none); OPERATING TEMPERATURE -55°C ~ 125°C -> (none); PACKAGE / CASE 0805 (2012 Metric) -> (none); PACKAGING Cut Tape (CT) -> (none); Part Number (none) -> GQM2195C1H101JB01D; QUANTITY AVAILABLE 5437 -> (none); TOLERANCE ±5% -> (none); UNIT PRICE (USD) 1.22 -> (none)
- C2: DATASHEET URL http://www.murata.com/~/media/webrenewal/support/library/ca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 -> (none); MANUFACTURER Murata Electronics North America -> (none); MANUFACTURER PART NUMBER GCJ21BR71A106KE01L -> (none); MOUNT Surface Mount, MLCC -> (none); OPERATING TEMPERATURE -55°C ~ 125°C -> (none); PACKAGE / CASE 0805 (2012 Metric) -> (none); PACKAGING Cut Tape (CT) -> (none); Part Number (none) -> GCJ21BR71A106KE01L; QUANTITY AVAILABLE 2702 -> (none); TOLERANCE ±10% -> (none); UNIT PRICE (USD) 0.56 -> (none)
- D1, D3: COLOR Red -> (none); FORWARD VOLTAGE 1.9V -> (none); LUMINOUS INTENSITY 60mcd -> (none); MANUFACTURER Wurth Elektronik -> (none); MANUFACTURER PART NUMBER 150080SS75000 -> (none); MOUNT Surface Mount -> (none); PACKAGING Cut Tape -> (none); Part Number (none) -> 150080SS75000
- D2: COLOR Green -> (none); FORWARD VOLTAGE 2.1V -> (none); LUMINOUS INTENSITY 12mcd -> (none); MANUFACTURER Vishay -> (none); MANUFACTURER PART NUMBER LTST-C171GKT -> (none); MOUNT Surface Mount -> (none); PACKAGING Tape and Reel -> (none); Part Number (none) -> LTST-C171GKT
- J1, J2, J5: COLOR White -> (none); MANUFACTURER Molex -> (none); MANUFACTURER PART NUMBER 22-05-3021 -> (none); MOUNT Through Hole -> (none); ORIENTATION Right Angle -> (none); PACKAGING Bulk -> (none); PITCH 2.54mm -> (none); Part Number (none) -> 22-05-3021
- J3, J4: DATASHEET URL https://www.molex.com/webdocs/datasheets/pdf/en-us/09012007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 -> (none); MANUFACTURER Molex -> (none); MANUFACTURER PART NUMBER 90120-0763 -> (none); MOUNT Board-To-Board Connector, C-Grid III 90120 Series, Through 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 -> (none); PITCH 2.54mm -> (none); Part Number (none) -> 90120-0763
- P1, P2: DATASHEET URL http://www.molex.com/pdm_docs/sd/022272041_sd.pdf -> (none); MANUFACTURER Molex -> (none); MANUFACTURER PART NUMBER 22-27-2041 -> (none); OPERATING TEMPERATURE 0degCto+75degC -> (none); Part Number (none) -> 22-27-2041
- P3: DATASHEET URL https://katalog.we-online.de/em/datasheet/6130xx11121.pdf -> (none); MANUFACTURER Wurth Elektronik -> (none); MANUFACTURER PART NUMBER 61300811121 -> (none); MOUNT Through Hole -> (none); OPERATING TEMPERATURE -40to105degC -> (none); ORIENTATION Vertical -> (none); PACKAGING Bag -> (none); PITCH 2.54mm -> (none); Part Number (none) -> 61300811121
- Q1, Q2: DATASHEET URL https://www.onsemi.com/pub/Collateral/FDN5632N_F085-D.PDF -> (none); MANUFACTURER Onsemi -> (none); MANUFACTURER PART NUMBER FDN5632N-F085 -> (none); Part Number (none) -> FDN5632N-F085
- R1, R2: DATASHEET URL https://industrial.panasonic.com/cdbs/www-data/pdf/RDA0000/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 -> (none); MANUFACTURER Panasonic Electronic Components -> (none); MANUFACTURER PART NUMBER ERJ-PB6D2000V -> (none); OPERATING TEMPERATURE -55°C ~ 155°C -> (none); PACKAGE / CASE 0805 (2012 Metric) -> (none); PACKAGING Cut Tape (CT) -> (none); POWER (WATTS) 0.25W, 1/4W -> (none); Part Number (none) -> ERJ-PB6D2000V; QUANTITY AVAILABLE 10000 -> (none); TOLERANCE ±0.5% -> (none); UNIT PRICE (USD) 0.04968 -> (none)
- R10: DATASHEET URL http://industrial.panasonic.com/www-cgi/jvcr13pz.cgi?E+PZ+3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 -> (none); MANUFACTURER Panasonic Electronic Components -> (none); MANUFACTURER PART NUMBER ERJ-6GEY0R00V -> (none); OPERATING TEMPERATURE -55°C ~ 155°C -> (none); PACKAGE / CASE 0805 (2012 Metric) -> (none); PACKAGING Cut Tape (CT) -> (none); POWER (WATTS) 0.125W, 1/8W -> (none); Part Number (none) -> ERJ-6GEY0R00V; QUANTITY AVAILABLE 1597627 -> (none); TOLERANCE Jumper -> (none); UNIT PRICE (USD) 0.00544 -> (none)
- R3, R4: DATASHEET URL http://industrial.panasonic.com/www-cgi/jvcr13pz.cgi?E+PZ+3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 -> (none); MANUFACTURER Panasonic Electronic Components -> (none); MANUFACTURER PART NUMBER ERJ-6ENF1002V -> (none); OPERATING TEMPERATURE -55°C ~ 155°C -> (none); PACKAGE / CASE 0805 (2012 Metric) -> (none); PACKAGING Cut Tape (CT) -> (none); POWER (WATTS) 0.125W, 1/8W -> (none); Part Number (none) -> ERJ-6ENF1002V; QUANTITY AVAILABLE 3985614 -> (none); TOLERANCE ±1% -> (none); UNIT PRICE (USD) 0.00729 -> (none)
- R7: DATASHEET URL http://industrial.panasonic.com/www-cgi/jvcr13pz.cgi?E+PZ+3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 -> (none); MANUFACTURER Panasonic Electronic Components -> (none); MANUFACTURER PART NUMBER ERJ-6ENF3090V -> (none); OPERATING TEMPERATURE -55°C ~ 155°C -> (none); PACKAGE / CASE 0805 (2012 Metric) -> (none); PACKAGING Cut Tape (CT) -> (none); POWER (WATTS) 0.125W, 1/8W -> (none); Part Number (none) -> ERJ-6ENF3090V; QUANTITY AVAILABLE 54759 -> (none); TOLERANCE ±1% -> (none); UNIT PRICE (USD) 0.00729 -> (none)
- R8: DATASHEET URL http://industrial.panasonic.com/www-cgi/jvcr13pz.cgi?E+PZ+3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 -> (none); MANUFACTURER Panasonic Electronic Components -> (none); MANUFACTURER PART NUMBER ERJ-6ENF76R8V -> (none); OPERATING TEMPERATURE -55°C ~ 155°C -> (none); PACKAGE / CASE 0805 (2012 Metric) -> (none); PACKAGING Cut Tape (CT) -> (none); POWER (WATTS) 0.125W, 1/8W -> (none); Part Number (none) -> ERJ-6ENF76R8V; QUANTITY AVAILABLE 23882 -> (none); TOLERANCE ±1% -> (none); UNIT PRICE (USD) 0.00729 -> (none)
- R9: DATASHEET URL http://industrial.panasonic.com/www-cgi/jvcr13pz.cgi?E+PZ+3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 -> (none); MANUFACTURER Panasonic Electronic Components -> (none); MANUFACTURER PART NUMBER ERJ-6ENF1400V -> (none); OPERATING TEMPERATURE -55°C ~ 155°C -> (none); PACKAGE / CASE 0805 (2012 Metric) -> (none); PACKAGING Cut Tape (CT) -> (none); POWER (WATTS) 0.125W, 1/8W -> (none); Part Number (none) -> ERJ-6ENF1400V; QUANTITY AVAILABLE 50700 -> (none); TOLERANCE ±1% -> (none); UNIT PRICE (USD) 0.00729 -> (none)
- U1: DATASHEET URL http://www.ti.com/lit/ds/symlink/msp430fr2355.pdf -> (none); MANUFACTURER Texas Instruments -> (none); MANUFACTURER PART NUMBER MSP430FR2355TPTR -> (none); Part Number (none) -> MSP430FR2355TPTR
- U2: DATASHEET URL http://www.st.com/internet/com/TECHNICAL_RESOURCES/TECHNICA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 -> (none); MANUFACTURER Onsemi -> (none); MANUFACTURER PART NUMBER LD1117S33TR -> (none); Part Number (none) -> LD1117S33TR
